Commit message: got something working for cartographer

File: b39vs_ws/src/hazmat_bringup/urdf/hazmat.urdf (robot description, URDF)
Before this commit: robot hazmat_robot, 3 links, 2 joints
Links:
- removed link world
- added link imu_link; collision sphere radius=0.025; visual sphere radius=0.025
- added link odom
Joints:
- added joint imu_joint: type fixed, parent central_frame, child imu_link, origin xyz=0.12 0 0.6 rpy=0 0 0
- joint base_joint: parent world -> odom

Commit message: added lidar link to urdf

File: b39vs_ws/src/hazmat_bringup/urdf/hazmat.urdf (robot description, URDF)
Before this commit: robot hazmat_robot, 4 links, 3 joints
Joints:
- added joint scan_joint: type fixed, parent central_frame, child imu_link, origin xyz=0.12 0 0.6 rpy=0 0 0

Commit message: fixed scan link

File: b39vs_ws/src/hazmat_bringup/urdf/hazmat.urdf (robot description, URDF)
Before this commit: robot hazmat_robot, 4 links, 4 joints
Links:
- added link scan_link; collision sphere radius=0.025; visual sphere radius=0.025
Joints:
- joint scan_joint: child imu_link -> scan_link

Commit message: modified caartographer config, changed hazmat_bringup build system to ament_python, added teleop launch

File: b39vs_ws/src/hazmat_bringup/urdf/hazmat.urdf (robot description, URDF)
Before this commit: robot hazmat_robot, 5 links, 4 joints
Links:
- removed link central_frame
- removed link imu_link
- added link base_link, mass 2.0; collision box size=0.3 0.3 0.1; visual box size=0.3 0.3 0.1
Joints:
- removed joint imu_joint
- joint base_joint: child central_frame -> base_link
- joint camera_joint: parent central_frame -> base_link
- joint scan_joint: parent central_frame -> base_link

Commit message: improved urdf to not use odom, added custom oak script to replace vendor launch file

File: b39vs_ws/src/hazmat_bringup/urdf/hazmat.urdf (robot description, URDF)
Before this commit: robot hazmat_robot, 4 links, 3 joints
Links:
- removed link odom
- added link base_footprint
- added link imu_link; visual sphere radius=0.025
- link base_link: mass 2.0 -> None; geometry visual box size=0.3 0.3 0.1
- link camera_link: geometry visual sphere radius=0.025
- link scan_link: geometry visual sphere radius=0.025
Joints:
- added joint imu_joint: type fixed, parent base_link, child imu_link, origin xyz=0.12 0 0.6 rpy=0 0 0
- joint base_joint: child base_link -> base_footprint; origin xyz=0 0 0 rpy=0 0 0 -> xyz=0 0 -0.035 rpy=0 0 0; parent odom -> base_link
- joint scan_joint: origin xyz=0.12 0 0.6 rpy=0 0 0 -> xyz=0.08 0 0.6 rpy=0 0 0

Commit message: added laserscan filter and fixed urdf

File: b39vs_ws/src/hazmat_bringup/urdf/hazmat.urdf (robot description, URDF)
Before this commit: robot hazmat_robot, 5 links, 4 joints
Joints:
- joint camera_joint: origin xyz=0.12 0 0.6 rpy=0 0 0 -> xyz=0.07 0 0.09 rpy=0 0 0
- joint imu_joint: origin xyz=0.12 0 0.6 rpy=0 0 0 -> xyz=0.07 0 0.09 rpy=0 0 0
- joint scan_joint: origin xyz=0.08 0 0.6 rpy=0 0 0 -> xyz=0.6 0 0.01 rpy=0 0 -1.5707

Commit message: all our changes frm this very long day

File: b39vs_ws/src/hazmat_bringup/urdf/hazmat.urdf (robot description, URDF)
Before this commit: robot hazmat_robot, 5 links, 4 joints
Joints:
- joint base_joint: child base_footprint -> base_link; origin xyz=0 0 -0.035 rpy=0 0 0 -> xyz=0 0 0.035 rpy=0 0 0; parent base_link -> base_footprint
- joint imu_joint: origin xyz=0.07 0 0.09 rpy=0 0 0 -> xyz=0.062 -0.038 0.089 rpy=3.142 1.571 0
- joint scan_joint: origin xyz=0.6 0 0.01 rpy=0 0 -1.5707 -> xyz=0.06 0 0.01 rpy=0 0 -1.571
